File: Mackie Onyx 1640 USB Option Card/Mackie Onyx 1640 USB Option Card.kicad_sch (KiCad schematic)
At the start: 1 part

Commit message: pcb design
Parts:
- added U1: XU316-1024-QF60B-C24, QFN_F60B-C24_XMO, symbol xmox:XU316-1024-QF60B-C24
- gave numbers to parts that had none: 1
Changed lines of the file:
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@@
 	(paper "A4")
+	(symbol
+		(lib_id "xmox:XU316-1024-QF60B-C24")
+		(at 93.98 78.74 0)
+		(unit 1)
+		(exclude_from_sim no)
+		(in_bom yes)
+		(on_board yes)
+		(dnp no)
+		(fields_autoplaced yes)
+		(property "Reference" "U1"
+			(at 121.92 68.58 0)
+			(effects
+				(font
+					(size 1.524 1.524)
+				)
+			)
+		)
+		(property "Value" "XU316-1024-QF60B-C24"
+			(at 121.92 71.12 0)
+			(effects
+				(font
+					(size 1.524 1.524)
+				)
+			)
+		)
+		(property "Footprint" "QFN_F60B-C24_XMO"
+			(at 93.98 78.74 0)
+			(effects
+				(font
+					(size 1.27 1.27)
+					(italic yes)
+				)
+				(hide yes)
+			)
+		)
+		(property "Datasheet" "XU316-1024-QF60B-C24"
+			(at 93.98 78.74 0)
+			(effects
+				(font
+					(size 1.27 1.27)
+					(italic yes)
+				)
+				(hide yes)
+			)
+		)
+		(property "Description" ""
+			(at 93.98 78.74 0)
+			(effects
+				(font
+					(size 1.27 1.27)
+				)
+				(hide yes)
+			)
+		)
+		(pin "6"
+		)
+		(pin "23"
+		)
+		(pin "25"
+		)
+		(pin "27"
+		)
+		(pin "22"
+		)
+		(pin "30"
+		)
+		(pin "1"
+		)
+		(pin "17"
+		)
+		(pin "4"
+		)
+		(pin "5"
+		)
+		(pin "7"
+		)
+		(pin "3"
+		)
+		(pin "9"
+		)
+		(pin "12"
+		)
+		(pin "13"
+		)
+		(pin "20"
+		)
+		(pin "2"
+		)
+		(pin "21"
+		)
+		(pin "15"
+		)
+		(pin "11"
+		)
+		(pin "14"
+		)
+		(pin "8"
+		)
+		(pin "10"
+		)
+		(pin "16"
+		)
+		(pin "18"
+		)
+		(pin "19"
+		)
+		(pin "24"
+		)
+		(pin "26"
+		)
+		(pin "28"
+		)
+		(pin "29"
+		)
+		(pin "55"
+		)
+		(pin "49"
+		)
+		(pin "43"
+		)
+		(pin "65"
+		)
+		(pin "39"
+		)
+		(pin "53"
+		)
+		(pin "54"
+		)
+		(pin "45"
+		)
+		(pin "41"
+		)
+		(pin "59"
+		)
+		(pin "61"
+		)
+		(pin "52"
+		)
+		(pin "48"
+		)
+		(pin "58"
+		)
+		(pin "56"
+		)
+		(pin "51"
+		)
+		(pin "46"
+		)
+		(pin "47"
+		)
+		(pin "31"
+		)
+		(pin "32"
+		)
+		(pin "64"
+		)
+		(pin "63"
+		)
+		(pin "60"
+		)
+		(pin "62"
+		)
+		(pin "57"
+		)
+		(pin "50"
+		)
+		(pin "44"
+		)
+		(pin "40"
+		)
+		(pin "42"
+		)
+		(pin "38"
+		)
+		(pin "37"
+		)
+		(pin "36"
+		)
+		(pin "35"
+		)
+		(pin "34"
+		)
+		(pin "33"
+		)
+		(instances
+			(project ""
+				(path "/c9b3cb63-7cfd-4f49-8501-d785ca0cd735"
+					(reference "U1")
+					(unit 1)
+				)
+			)
+		)
+	)
 	(symbol
 		(lib_id "Connector_Generic:Conn_02x17_Odd_Even")
@@
 		(dnp no)
 		(fields_autoplaced yes)
-		(property "Reference" "J?"
+		(property "Reference" "J1"
 			(at 229.87 63.5 0)
 			(effects
@@
 			(project ""
 				(path "/c9b3cb63-7cfd-4f49-8501-d785ca0cd735"
-					(reference "J?")
+					(reference "J1")
 					(unit 1)
 				)

Commit message: PCB connector documentation added
Parts:
- added U2, U3, U4: CS5368-CQZ, adc:CIR-LQFP-48, symbol adc:CS5368-CQZ
Connections:
- net CH1_DIREKT_OUT: now reaches J1.1 (Pin_1)
- net CH10_DIREKT_OUT: now reaches J1.10 (Pin_10)
- net CH11_DIREKT_OUT: now reaches J1.11 (Pin_11)
- net CH12_DIREKT_OUT: now reaches J1.12 (Pin_12)
- net CH13_DIREKT_OUT: now reaches J1.13 (Pin_13)
- net CH14_DIREKT_OUT: now reaches J1.14 (Pin_14)
- net CH15_DIREKT_OUT: now reaches J1.15 (Pin_15)
- net CH16_DIREKT_OUT: now reaches J1.16 (Pin_16)
- net GND: now reaches J1.17 (Pin_17)
- net GND: now also J1.18 (Pin_18), J1.21 (Pin_21), J1.22 (Pin_22)
- net L_SEND: now reaches J1.19 (Pin_19)
- net CH2_DIREKT_OUT: now reaches J1.2 (Pin_2)
- net R_SEND: now reaches J1.20 (Pin_20)
- net L_OUT: now reaches J1.23 (Pin_23)
- net R_OUT: now reaches J1.24 (Pin_24)
- net +15V: now reaches J1.25 (Pin_25)
- net -15V: now reaches J1.27 (Pin_27)
- net Earth: now reaches J1.29 (Pin_29)
- net Earth: now also J1.30 (Pin_30), J1.31 (Pin_31)
- net CH3_DIREKT_OUT: now reaches J1.3 (Pin_3)
- net +5V: now reaches J1.33 (Pin_33)
- net CH4_DIREKT_OUT: now reaches J1.4 (Pin_4)
- net CH5_DIREKT_OUT: now reaches J1.5 (Pin_5)
- net CH6_DIREKT_OUT: now reaches J1.6 (Pin_6)
- net CH7_DIREKT_OUT: now reaches J1.7 (Pin_7)
- net CH8_DIREKT_OUT: now reaches J1.8 (Pin_8)
- net CH9_DIREKT_OUT: now reaches J1.9 (Pin_9)
Other:
- title: (none) -> Connector
- moved on the sheet: J1, U1
