File: Mackie Onyx 1640 USB Option Card/Mackie Onyx 1640 USB Option Card.kicad_sch (KiCad schematic)
At the start: 5 parts, among them J1 Conn_02x17_Odd_Even, U1 XU316-1024-QF60B-C24, U2 CS5368-CQZ, U3 CS5368-CQZ, U4 CS5368-CQZ

Commit message: MO1640 USB Schematic work
Parts:
- removed J1: Conn_02x17_Odd_Even, Connector_IDC:IDC-Header_2x17_P2.54mm_Latch_Horizontal, symbol Connector_Generic:Conn_02x17_Odd_Even
- removed U1: XU316-1024-QF60B-C24, QFN_F60B-C24_XMO, symbol xmox:XU316-1024-QF60B-C24
- removed U2, U3, U4: CS5368-CQZ, adc:CIR-LQFP-48, symbol adc:CS5368-CQZ
Other:
- added sheet Connector (Connector.kicad_sch)
- title: Connector -> MackieOnyx 1640 USB Option Card
