File: Mackie Onyx 1640 USB Option Card/Mackie Onyx 1640 USB Option Card.kicad_sch (KiCad schematic)
At the start: 3 parts, among them SW1 SW_Push, U1 XU316-1024-QF60B-C24, Y1 24MHz Crystal

Commit message: addet audio codec
addet TAC5212 footprint to projekt library
addet ADC_DAC page for Main Mix out L&R, Interface IN R&L
Other:
- added sheet ADC_DAC (ADC_DAC.kicad_sch)
Changed lines of the file:
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@@
+		)
+	)
+	(sheet
+		(at 218.44 58.42)
+		(size 22.86 16.51)
+		(exclude_from_sim no)
+		(in_bom yes)
+		(on_board yes)
+		(dnp no)
+		(fields_autoplaced yes)
+		(stroke
+			(width 0.1524)
+			(type solid)
+		)
+		(fill
+			(color 0 0 0 0.0000)
+		)
+		(property "Sheetname" "ADC_DAC"
+			(at 218.44 57.7084 0)
+			(effects
+				(font
+					(size 1.27 1.27)
+				)
+				(justify left bottom)
+			)
+		)
+		(property "Sheetfile" "ADC_DAC.kicad_sch"
+			(at 218.44 75.5146 0)
+			(effects
+				(font
+					(size 1.27 1.27)
+				)
+				(justify left top)
+			)
+		)
+		(pin "IN2" input
+			(at 241.3 63.5 0)
+			(effects
+				(font
+					(size 1.27 1.27)
+				)
+				(justify right)
+			)
+		)
+		(pin "OUT1" output
+			(at 241.3 66.04 0)
+			(effects
+				(font
+					(size 1.27 1.27)
+				)
+				(justify right)
+			)
+		)
+		(pin "OUT2" output
+			(at 241.3 68.58 0)
+			(effects
+				(font
+					(size 1.27 1.27)
+				)
+				(justify right)
+			)
+		)
+		(pin "IN1" input
+			(at 241.3 60.96 0)
+			(effects
+				(font
+					(size 1.27 1.27)
+				)
+				(justify right)
+			)
+		)
+		(instances
+			(project "Mackie Onyx 1640 USB Option Card"
+				(path "/c9b3cb63-7cfd-4f49-8501-d785ca0cd735"
+					(page "8")
+				)
+			)
 		)
 	)
